Commit message: change_from_stl_to_boxes_but_motion_direction_is_reversed

File: urdf/common_properties.xacro (robot description, xacro)
@@ -1,4 +1,10 @@
 <?xml version="1.0"?>
 <robot xmlns:xacro="http://www.ros.org/wiki/xacro">
+    <material name="blue">
+        <color rgba="0 0 0.5 1" />
+    </material>
+    <material name="grey">
+        <color rgba="0.5 0.5 0.5 1" />
+    </material>
     <xacro:macro name="box_inertia" params="m l w h xyz rpy">
         <inertial>

File: urdf/imu.xacro (robot description, xacro)
@@ -26,5 +26,5 @@
   </link>
   <joint name="imu_joint" type="fixed">
-    <origin xyz="0.065 0.012 0.043" rpy="0 0 0" />
+    <origin xyz="0.065 0.012 0.027" rpy="0 0 0" />
     <parent link="upper_link" />
     <child link="imu_link" />

File: urdf/lidar.xacro (robot description, xacro)
@@ -36,5 +36,5 @@
                 <range>
                     <min>0.3</min>
-                    <max>4</max>
+                    <max>20</max>
                 </range>
             </ray>

File: urdf/robitcubebot_base.xacro (robot description, xacro)
@@ -1,171 +1,104 @@
 <?xml version="1.0"?>
-<robot name="robitcubebot" xmlns:xacro="http://ros.org/wiki/xacro">
-  <xacro:include filename="common_properties.xacro" />
-  <link name="base_footprint"/>
-  <!-- Define robot properties -->
-  <xacro:property name="base_length" value="0.317" />
-  <xacro:property name="base_width" value="0.212" />
-  <xacro:property name="base_height" value="0.0446" />
-  <xacro:property name="wheel_radius" value="0.0325" />
-  <xacro:property name="wheel_length" value="0.025" />
-  <link name="base_link">
-    <xacro:box_inertia m="0.6" l="${2*base_length}" w="${2*base_width}" h="${2*base_height}"
+<robot xmlns:xacro="http://www.ros.org/wiki/xacro">
+    <xacro:property name="base_length" value="0.317" />
+    <xacro:property name="base_width" value="0.212" />
+    <xacro:property name="base_height" value="0.0446" />
+    <xacro:property name="upper_length" value="0.317" />
+    <xacro:property name="upper_width" value="0.212" />
+    <xacro:property name="upper_height" value="0.0423" />
+    <xacro:property name="wheel_radius" value="0.0325" />
+    <xacro:property name="wheel_length" value="0.028" />
+    <xacro:property name="to_wheel_center" value="0.07" />
+    <link name="base_footprint" />
+    <link name="base_link">
+        <visual>
+            <geometry>
+                <box size="${base_length} ${base_width} ${base_height}" />
+            </geometry>
+            <origin xyz="0 0 ${base_height / 2.0}" rpy="0 0 0" />
+          <material name="blue" />
+        </visual>
+        <collision>
+            <geometry>
+                <box size="${base_length} ${base_width} ${base_height}" />
+            </geometry>
+            <origin xyz="0 0 ${base_height / 2.0}" rpy="0 0 0" />
+        </collision>
+        <xacro:box_inertia m="5.0" l="${2*base_length}" w="${2*base_width}" h="${2*base_height}"
                            xyz="0 0 ${base_height / 2.0}" rpy="0 0 0" />
-    <visual>
-      <origin xyz="-${base_length / 2.0} -${base_width / 2.0} 0" rpy="0 0 0" />
-      <geometry>
-        <mesh filename="package://robitcubebot_description/meshes/base_link.STL" scale="0.001 0.001 0.001" />
-      </geometry>
-      <material name="black">
-          <color rgba="0.1 0.1 0.1 1" />
-      </material>
-    </visual>
-    <collision>
-      <origin xyz="0 0 0.1" rpy="0 0 0" />
-      <geometry>
-        <box size="${base_length} ${base_width} ${base_height}" />
-      </geometry>
-    </collision>
-  </link>
-  <!-- Define joints -->
-  <joint name="base_joint" type="fixed">
-    <parent link="base_footprint"/>
-    <child link="base_link" />
-    <origin xyz="0 0 0" rpy="0 0 0"/>
-  </joint>
-  <!-- Wheels -->
-  <link name="front_wheel_right_link">
-    <inertial>
-      <origin xyz="0 -0.014 0" rpy="0 0 0" />
-      <mass value="0.0530086090966721" />
-      <inertia ixx="1.88176298336665E-05" ixy="-4.8444933029987E-10" ixz="1.88163708851143E-08"
-               iyy="3.11510738647764E-05" iyz="-6.93560663069607E-11"
-               izz="1.8801969558182E-05" />
-    </inertial>
-    <visual>
-      <origin xyz="0 0 0" rpy="1.57 0 0" />
-      <geometry>
-        <mesh filename="package://robitcubebot_description/meshes/wheel_right_link.STL" />
-      </geometry>
-    </visual>
-    <collision>
-      <origin xyz="0 -0.015 0" rpy="1.57 0 0" />
-      <geometry>
-        <sphere radius="0.033"/>
-      </geometry>
-    </collision>
-  </link>
-  <joint name="front_wheel_right_joint" type="continuous">
-    <origin xyz="-${base_width / 1.8} -${base_width / 2.1} ${wheel_radius}" rpy="0 0 0" />
-    <parent link="base_link" />
-    <child link="front_wheel_right_link" />
-    <axis xyz="0 -1 0" />
-  </joint>
-  <link
-    name="front_wheel_left_link">
-    <inertial>
-      <origin xyz="0 0.014 0" rpy="0 0 0" />
-      <mass value="0.0530086043217644" />
-      <inertia ixx="1.8792911368909E-05"  ixy="3.31256392204584E-10" ixz="-1.14082001662767E-08"
-               iyy="3.11510738759073E-05" iyz="-3.60499245082192E-10"
-               izz="1.88266886146847E-05" />
-    </inertial>
-    <visual>
-      <origin xyz="0 0 0" rpy="-1.57 0 0" />
-      <geometry>
-        <mesh filename="package://robitcubebot_description/meshes/wheel_left_link.STL" />
-      </geometry>
-    </visual>
-    <collision>
-      <origin xyz="0 0.015 0" rpy="-1.57 0 0" />
-      <geometry>
-        <sphere radius="0.033"/>
-      </geometry>
-    </collision>
-  </link>
-  <joint name="front_wheel_left_joint" type="continuous">
-    <origin xyz="-${base_width / 1.8} ${base_width / 2.1} ${wheel_radius}" rpy="0 0 0" />
-    <parent link="base_link" />
-    <child link="front_wheel_left_link" />
-    <axis xyz="0 -1 0" />
-  </joint>
-  <link name="back_wheel_right_link">
-    <inertial>
-      <origin xyz="0 -0.014 0" rpy="0 0 0" />
-      <mass value="0.0530086090966721" />
-      <inertia ixx="1.88176298336665E-05" ixy="-4.8444933029987E-10" ixz="1.88163708851143E-08"
-               iyy="3.11510738647764E-05" iyz="-6.93560663069607E-11"
-               izz="1.8801969558182E-05" />
-    </inertial>
-    <visual>
-      <origin xyz="0 0 0" rpy="1.57 0 0" />
-      <geometry>
-        <mesh filename="package://robitcubebot_description/meshes/wheel_right_link.STL" />
-      </geometry>
-    </visual>
-    <collision>
-      <origin xyz="0 -0.015 0" rpy="1.57 0 0" />
-      <geometry>
-        <sphere radius="0.033"/>
-      </geometry>
-    </collision>
-  </link>
-  <joint name="back_wheel_right_joint" type="continuous">
-    <origin xyz="${base_width / 1.8} -${base_width / 2.1} ${wheel_radius}" rpy="0 0 0" />
-    <parent link="base_link" />
-    <child link="back_wheel_right_link" />
-    <axis xyz="0 -1 0" />
-  </joint>
-  <link
-    name="back_wheel_left_link">
-    <inertial>
-      <origin xyz="0 0.014 0" rpy="0 0 0" />
-      <mass value="0.0530086043217644" />
-      <inertia ixx="1.8792911368909E-05"  ixy="3.31256392204584E-10" ixz="-1.14082001662767E-08"
-               iyy="3.11510738759073E-05" iyz="-3.60499245082192E-10"
-               izz="1.88266886146847E-05" />
-    </inertial>
-    <visual>
-      <origin xyz="0 0 0" rpy="-1.57 0 0" />
-      <geometry>
-        <mesh filename="package://robitcubebot_description/meshes/wheel_left_link.STL" />
-      </geometry>
-    </visual>
-    <collision>
-      <origin xyz="0 0.015 0" rpy="-1.57 0 0" />
-      <geometry>
-        <sphere radius="0.033"/>
-      </geometry>
-    </collision>
-  </link>
-  <joint name="back_wheel_left_joint" type="continuous">
-    <origin xyz="${base_width / 1.8} ${base_width / 2.1} ${wheel_radius}" rpy="0 0 0" />
-    <parent link="base_link" />
-    <child link="back_wheel_left_link" />
-    <axis xyz="0 -1 0" />
-  </joint>
-  <link name="upper_link">
-    <xacro:box_inertia m="0.6" l="${2*base_length}" w="${2*base_width}" h="${2*base_height}"
+    </link>
+    <link name="upper_link">
+        <visual>
+            <geometry>
+                <box size="${upper_length} ${upper_width} ${upper_height}" />
+            </geometry>
+            <origin xyz="0 0 0" rpy="0 0 0" />
+            <material name="grey" />
+        </visual>
+        <collision>
+            <geometry>
+                <box size="${base_length} ${base_width} ${base_height}" />
+            </geometry>
+            <origin xyz="0 0 ${upper_height / 2.0}" rpy="0 0 0" />
+        </collision>
+        <xacro:box_inertia m="5.0" l="${2*base_length}" w="${2*base_width}" h="${2*base_height}"
                            xyz="0 0 ${base_height / 2.0}" rpy="0 0 0" />
-    <visual>
-      <origin xyz="-${base_length / 1.75} -0.165 0" rpy="0 0 0" />
-      <geometry>
-        <mesh filename="package://robitcubebot_description/meshes/upper_link.STL" scale="0.001 0.001 0.001" />
-      </geometry>
-      <material name="black">
-        <color rgba="0.1 0.1 0.1 1" />
-      </material>
-    </visual>
-    <collision>
-      <origin xyz="0 0 ${base_height}" rpy="0 0 0" />
-      <geometry>
-        <box size="${base_length} ${base_width} ${base_height}" />
-      </geometry>
-    </collision>
-  </link>
-  <joint name="upper_joint" type="fixed">
-    <parent link="base_link"/>
-    <child link="upper_link" />
-    <origin xyz="0 0 ${base_height}" rpy="0 0 0"/>
-  </joint>
+    </link>
+    <xacro:macro name="wheel_link" params="prefix">
+        <link name="${prefix}_wheel_link">
+            <visual>
+                <geometry>
+                    <cylinder radius="${wheel_radius}" length="${wheel_length}" />
+                </geometry>
+                <origin xyz="0 0 0" rpy="${pi / 2.0} 0 0" />
+                <material name="grey" />
+            </visual>
+            <collision>
+                <geometry>
+                    <cylinder radius="${wheel_radius}" length="${wheel_length}" />
+                </geometry>
+                <origin xyz="0 0 0" rpy="${pi / 2.0} 0 0" />
+            </collision>
+            <xacro:cylinder_inertia m="1.0" r="${2*wheel_radius}" h="${2*wheel_length}"
+                                    xyz="0 0 0" rpy="${pi / 2.0} 0 0" />
+        </link>
+    </xacro:macro>
+    <xacro:wheel_link prefix="front_right" />
+    <xacro:wheel_link prefix="front_left" />
+    <xacro:wheel_link prefix="back_right" />
+    <xacro:wheel_link prefix="back_left" />
+    <joint name="base_joint" type="fixed">
+        <parent link="base_footprint" />
+        <child link="base_link" />
+        <origin xyz="0 0 ${wheel_radius}" rpy="0 0 0"/>
+    </joint>
+    <joint name="upper_joint" type="fixed">
+        <parent link="base_link" />
+        <child link="upper_link" />
+        <origin xyz="0 0 ${base_height+base_height / 2.0}" rpy="0 0 0"/>
+    </joint>
+    <joint name="front_wheel_right_joint" type="continuous">
+        <parent link="base_link" />
+        <child link="front_right_wheel_link" />
+        <origin xyz="${-base_length / 2.7} ${-(base_width + wheel_length) / 2.0} 0" rpy="0 0 0" />
+        <axis xyz="0 1 0" />
+    </joint>
+    <joint name="front_wheel_left_joint" type="continuous">
+        <parent link="base_link" />
+        <child link="front_left_wheel_link" />
+        <origin xyz="${-base_length / 2.7} ${(base_width + wheel_length) / 2.0} 0" rpy="0 0 0" />
+        <axis xyz="0 1 0" />
+    </joint>
+    <joint name="back_wheel_right_joint" type="continuous">
+        <parent link="base_link" />
+        <child link="back_right_wheel_link" />
+        <origin xyz="${base_length / 2.7} ${-(base_width + wheel_length) / 2.0} 0" rpy="0 0 0" />
+        <axis xyz="0 1 0" />
+    </joint>
+    <joint name="back_wheel_left_joint" type="continuous">
+        <parent link="base_link" />
+        <child link="back_left_wheel_link" />
+        <origin xyz="${base_length / 2.7} ${(base_width + wheel_length) / 2.0} 0" rpy="0 0 0" />
+        <axis xyz="0 1 0" />
+    </joint>
 </robot>
