Commit message: change_imu_to_baselink_but_not_working

File: urdf/imu.xacro (robot description, xacro)
@@ -26,6 +26,6 @@
   </link>
   <joint name="imu_joint" type="fixed">
-    <origin xyz="0.065 0.012 0.043" rpy="0 0 0" />
-    <parent link="upper_link" />
+    <origin xyz="0 0 0" rpy="0 0 0" />
+    <parent link="base_link" />
     <child link="imu_link" />
     <axis xyz="0 0 0" />

File: urdf/robitcubebot_base.xacro (robot description, xacro)
@@ -32,5 +32,5 @@
     <parent link="base_footprint"/>
     <child link="base_link" />
-    <origin xyz="0 0 0" rpy="0 0 0"/>
+    <origin xyz="0 0 0" rpy="0 0 3.14"/>
   </joint>
   <!-- Wheels -->
