Commit message: wheels_pos

File: urdf/lidar.xacro (robot description, xacro)
@@ -4,10 +4,10 @@
         <parent link="upper_link"/>
         <child link="laser_frame"/>
-        <origin xyz="-${base_length /2.5} 0.005 ${base_height-0.01}" rpy="0 0 0"/>
+        <origin xyz="-0.1 0.005 ${base_height}" rpy="0 0 0"/>
     </joint>
     <link name="laser_frame">
         <visual>
             <geometry>
-                <cylinder radius="0.034" length="0.03"/>
+                <cylinder radius="0.0508" length="0.055"/>
             </geometry>
         </visual>
@@ -50,5 +50,5 @@
                                     xyz="0 0 0" rpy="${pi / 2.0} 0 0" />
     </link-->
-  <gazebo reference="laser_frame">
+  <!--gazebo reference="laser_frame">
     <material>Gazebo/FlatBlack</material>
     <sensor type="ray" name="lds_lfcd_sensor">
@@ -81,4 +81,32 @@
       </plugin>
     </sensor>
-  </gazebo>
+  </gazebo-->
+  <gazebo reference="laser_frame">
+        <material>Gazebo/Black</material>
+        <sensor name="laser" type="ray">
+            <pose> 0 0 0 0 0 0 </pose>
+            <visualize>false</visualize>
+            <update_rate>10</update_rate>
+            <ray>
+                <scan>
+                    <horizontal>
+                        <samples>360</samples>
+                        <min_angle>-3.14</min_angle>
+                        <max_angle>3.14</max_angle>
+                    </horizontal>
+                </scan>
+                <range>
+                    <min>0.3</min>
+                    <max>12</max>
+                </range>
+            </ray>
+            <plugin name="laser_controller" filename="libgazebo_ros_ray_sensor.so">
+                <ros>
+                    <argument>~/out:=scan</argument>
+                </ros>
+                <output_type>sensor_msgs/LaserScan</output_type>
+                <frame_name>laser_frame</frame_name>
+            </plugin>
+        </sensor>
+    </gazebo>
 </robot>

File: urdf/robitcubebot_base.xacro (robot description, xacro)
@@ -32,5 +32,6 @@
     <parent link="base_footprint"/>
     <child link="base_link" />
-    <origin xyz="0 0 ${wheel_radius}" rpy="0 0 3.14"/>
+    <!--origin xyz="0 0 ${wheel_radius}" rpy="0 0 3.14"/-->
+    <origin xyz="0 0 0" rpy="0 0 3.14"/>
   </joint>
   <!-- Wheels -->
@@ -50,5 +51,6 @@
     </visual>
     <collision>
-      <origin xyz="0 -0.015 0" rpy="1.57 0 0" />
+      <!--origin xyz="0 -0.015 0" rpy="1.57 0 0" /-->
+      <origin xyz="0 0 0" rpy="1.57 0 0" />
       <geometry>
         <sphere radius="0.033"/>
@@ -78,5 +80,6 @@
     </visual>
     <collision>
-      <origin xyz="0 0.015 0" rpy="-1.57 0 0" />
+      <!--origin xyz="0 0.015 0" rpy="-1.57 0 0" /-->
+      <origin xyz="0 0 0" rpy="-1.57 0 0" />
       <geometry>
         <sphere radius="0.033"/>
@@ -85,5 +88,5 @@
   </link>
   <joint name="front_wheel_left_joint" type="continuous">
-    <origin xyz="-${base_width / 1.8} ${base_width / 2.1} ${wheel_radius}" rpy="0 0 0" />
+    <origin xyz="-${base_width / 1.8} ${base_width / 2} ${wheel_radius}" rpy="0 0 0" />
     <parent link="base_link" />
     <child link="front_wheel_left_link" />
@@ -105,5 +108,6 @@
     </visual>
     <collision>
-      <origin xyz="0 -0.015 0" rpy="1.57 0 0" />
+      <!--origin xyz="0 -0.015 0" rpy="1.57 0 0" /-->
+      <origin xyz="0 0 0" rpy="1.57 0 0" />
       <geometry>
         <sphere radius="0.033"/>
@@ -111,10 +115,9 @@
     </collision>
   </link>
-  <joint name="back_wheel_right_joint" type="revolute">
+  <joint name="back_wheel_right_joint" type="fixed">
     <origin xyz="${base_width / 1.8} -${base_width / 2.1} ${wheel_radius}" rpy="0 0 0" />
     <parent link="base_link" />
     <child link="back_wheel_right_link" />
     <axis xyz="0 -1 0" />
-    <limit effort="10" velocity="10" lower="-1.57" upper="1.57"/>
   </joint>
   <link
@@ -134,5 +137,6 @@
     </visual>
     <collision>
-      <origin xyz="0 0.015 0" rpy="-1.57 0 0" />
+      <!--origin xyz="0 0.015 0" rpy="-1.57 0 0" /-->
+      <origin xyz="0 0 0" rpy="-1.57 0 0" />
       <geometry>
         <sphere radius="0.033"/>
@@ -140,10 +144,9 @@
     </collision>
   </link>
-  <joint name="back_wheel_left_joint" type="revolute">
-    <origin xyz="${base_width / 1.8} ${base_width / 2.1} ${wheel_radius}" rpy="0 0 0" />
+  <joint name="back_wheel_left_joint" type="fixed">
+    <origin xyz="${base_width / 1.8} ${base_width / 2} ${wheel_radius}" rpy="0 0 0" />
     <parent link="base_link" />
     <child link="back_wheel_left_link" />
     <axis xyz="0 -1 0" />
-    <limit effort="10" velocity="10" lower="-1.57" upper="1.57"/>
   </joint>
   <link name="upper_link">

Commit message: lidar_and_motion_adjustment

File: urdf/lidar.xacro (robot description, xacro)
@@ -4,5 +4,5 @@
         <parent link="upper_link"/>
         <child link="laser_frame"/>
-        <origin xyz="-${base_length /2.5} 0.005 ${base_height-0.01}" rpy="0 0 0"/>
+        <origin xyz="-${base_length /2.5} 0.005 0.06" rpy="0 0 0"/>
     </joint>
     <link name="laser_frame">
@@ -50,35 +50,31 @@
                                     xyz="0 0 0" rpy="${pi / 2.0} 0 0" />
     </link-->
-  <gazebo reference="laser_frame">
-    <material>Gazebo/FlatBlack</material>
-    <sensor type="ray" name="lds_lfcd_sensor">
-      <pose>0 0 0 0 0 0</pose>
-      <visualize>true</visualize>
-      <update_rate>5</update_rate>
-      <ray>
-        <scan>
-          <horizontal>
-            <samples>360</samples>
-            <resolution>1</resolution>
-            <min_angle>0.0</min_angle>
-            <max_angle>6.28319</max_angle>
-          </horizontal>
-        </scan>
-        <range>
-          <min>0.120</min>
-          <max>3.5</max>
-          <resolution>0.015</resolution>
-        </range>
-        <noise>
-          <type>gaussian</type>
-          <mean>0.0</mean>
-          <stddev>0.01</stddev>
-        </noise>
-      </ray>
-      <plugin name="gazebo_ros_lds_lfcd_controller" filename="libgazebo_ros_laser.so">
-        <topicName>scan</topicName>
-        <frameName>laser_frame</frameName>
-      </plugin>
-    </sensor>
-  </gazebo>
+    <!--gazebo reference="laser_frame">
+        <material>Gazebo/Red</material>
+        <sensor name="laser" type="ray">
+            <pose> 0 0 0 0 0 0 </pose>
+            <visualize>true</visualize>
+            <update_rate>10</update_rate>
+            <ray>
+                <scan>
+                    <horizontal>
+                        <samples>360</samples>
+                        <min_angle>-3.14</min_angle>
+                        <max_angle>3.14</max_angle>
+                    </horizontal>
+                </scan>
+                <range>
+                    <min>0.3</min>
+                    <max>12</max>
+                </range>
+            </ray>
+            <plugin name="laser_controller" filename="libgazebo_ros_ray_sensor.so">
+                <ros>
+                    <argument>~/out:=scan</argument>
+                </ros>
+                <output_type>sensor_msgs/LaserScan</output_type>
+                <frame_name>laser_frame</frame_name>
+            </plugin>
+        </sensor>
+    </gazebo-->
 </robot>

File: urdf/lift.xacro (robot description, xacro)
@@ -62,4 +62,6 @@
     <axis xyz="0 0 1" rpy="0 0 0"/>
     <limit effort="10000.0" lower="-0.05" upper="-0.035" velocity="0.2"/>
+    <dynamics damping="0.1" friction="0.1"/>
+    <hardwareInterface>hardware_interface/VelocityJointInterface</hardwareInterface>
   </joint>
 </robot>

File: urdf/robitcubebot_base.xacro (robot description, xacro)
@@ -32,5 +32,5 @@
     <parent link="base_footprint"/>
     <child link="base_link" />
-    <origin xyz="0 0 ${wheel_radius}" rpy="0 0 3.14"/>
+    <origin xyz="0 0 0" rpy="0 0 0"/>
   </joint>
   <!-- Wheels -->
@@ -111,10 +111,9 @@
     </collision>
   </link>
-  <joint name="back_wheel_right_joint" type="revolute">
+  <joint name="back_wheel_right_joint" type="continuous">
     <origin xyz="${base_width / 1.8} -${base_width / 2.1} ${wheel_radius}" rpy="0 0 0" />
     <parent link="base_link" />
     <child link="back_wheel_right_link" />
     <axis xyz="0 -1 0" />
-    <limit effort="10" velocity="10" lower="-1.57" upper="1.57"/>
   </joint>
   <link
@@ -140,10 +139,9 @@
     </collision>
   </link>
-  <joint name="back_wheel_left_joint" type="revolute">
+  <joint name="back_wheel_left_joint" type="continuous">
     <origin xyz="${base_width / 1.8} ${base_width / 2.1} ${wheel_radius}" rpy="0 0 0" />
     <parent link="base_link" />
     <child link="back_wheel_left_link" />
     <axis xyz="0 -1 0" />
-    <limit effort="10" velocity="10" lower="-1.57" upper="1.57"/>
   </joint>
   <link name="upper_link">

File: urdf/robitcubebot_gazebo.xacro (robot description, xacro)
@@ -16,5 +16,5 @@
     </joint>
   </transmission>
-  <!--transmission name="back_right_wheel_transmission">
+  <transmission name="back_right_wheel_transmission">
     <plugin>transmission_interface/SimpleTransmission</plugin>
     <actuator name="back_wheel_right_motor" role="back_actuator_right"/>
@@ -29,5 +29,5 @@
       <mechanical_reduction>1.0</mechanical_reduction>
     </joint>
-  </transmission-->
+  </transmission>
   <!-- Wheels -->
   <gazebo reference="front_wheel_left_link">

Commit message: lidar_taha

File: urdf/lidar.xacro (robot description, xacro)
@@ -2,7 +2,7 @@
 <robot xmlns:xacro="http://www.ros.org/wiki/xacro" >
     <joint name="laser_joint" type="fixed">
-        <parent link="upper_link"/>
+        <parent link="base_link"/>
         <child link="laser_frame"/>
-        <origin xyz="-${base_length /2.5} 0.005 0.06" rpy="0 0 0"/>
+        <origin xyz="-${base_length /2.5} 0.005 0.1" rpy="0 0 0"/>
     </joint>
     <link name="laser_frame">
@@ -20,35 +20,5 @@
                                     xyz="0 0 0" rpy="${pi / 2.0} 0 0" />
     </link>
-    <!--joint name="laser_joint_down" type="fixed">
-        <parent link="upper_link"/>
-        <child link="laser_frame_down"/>
-        <origin xyz="-0.152  -0.012 0" rpy="0 0 0"/>
-    </joint>
-    <link name="laser_frame">
-    </link>
-    <joint name="laser_joint" type="fixed">
-        <parent link="laser_frame_down"/>
-        <child link="laser_frame"/>
-        <origin xyz="0 0 -0.01" rpy="0 0 0"/>
-    </joint>
-    <link name="laser_frame_down">
-        <visual>
-            <origin xyz="0.003 0.12 -0.043" rpy="1.57 0 0"/>
-            <geometry>
-                <mesh filename="package://robitcubebot_description/meshes/lidar.STL" scale="0.001 0.001 0.001" />
-            </geometry>
-            <material name="black">
-                <color rgba="0.1 0.1 0.1 1" />
-            </material>
-        </visual>
-        <collision>
-            <geometry>
-                <mesh filename="package://robitcubebot_description/meshes/lidar.STL" scale="0.001 0.001 0.001" />
-            </geometry>
-        </collision>
-        <xacro:cylinder_inertia m="1.0" r="${2*0.05}" h="${2*0.04}"
-                                    xyz="0 0 0" rpy="${pi / 2.0} 0 0" />
-    </link-->
-    <!--gazebo reference="laser_frame">
+    <gazebo reference="laser_frame">
         <material>Gazebo/Red</material>
         <sensor name="laser" type="ray">
@@ -66,5 +36,5 @@
                 <range>
                     <min>0.3</min>
-                    <max>12</max>
+                    <max>4</max>
                 </range>
             </ray>
@@ -77,4 +47,4 @@
             </plugin>
         </sensor>
-    </gazebo-->
+    </gazebo>
 </robot>

Commit message: add lift control and edit lidar simulation in gazebo

File: urdf/lidar.xacro (robot description, xacro)
@@ -2,5 +2,5 @@
 <robot xmlns:xacro="http://www.ros.org/wiki/xacro" >
     <joint name="laser_joint" type="fixed">
-        <parent link="upper_link"/>
+        <parent link="base_link"/>
         <child link="laser_frame"/>
         <origin xyz="-${base_length /2.5} 0.005 0.06" rpy="0 0 0"/>
@@ -20,35 +20,5 @@
                                     xyz="0 0 0" rpy="${pi / 2.0} 0 0" />
     </link>
-    <!--joint name="laser_joint_down" type="fixed">
-        <parent link="upper_link"/>
-        <child link="laser_frame_down"/>
-        <origin xyz="-0.152  -0.012 0" rpy="0 0 0"/>
-    </joint>
-    <link name="laser_frame">
-    </link>
-    <joint name="laser_joint" type="fixed">
-        <parent link="laser_frame_down"/>
-        <child link="laser_frame"/>
-        <origin xyz="0 0 -0.01" rpy="0 0 0"/>
-    </joint>
-    <link name="laser_frame_down">
-        <visual>
-            <origin xyz="0.003 0.12 -0.043" rpy="1.57 0 0"/>
-            <geometry>
-                <mesh filename="package://robitcubebot_description/meshes/lidar.STL" scale="0.001 0.001 0.001" />
-            </geometry>
-            <material name="black">
-                <color rgba="0.1 0.1 0.1 1" />
-            </material>
-        </visual>
-        <collision>
-            <geometry>
-                <mesh filename="package://robitcubebot_description/meshes/lidar.STL" scale="0.001 0.001 0.001" />
-            </geometry>
-        </collision>
-        <xacro:cylinder_inertia m="1.0" r="${2*0.05}" h="${2*0.04}"
-                                    xyz="0 0 0" rpy="${pi / 2.0} 0 0" />
-    </link-->
-    <!--gazebo reference="laser_frame">
+    <gazebo reference="laser_frame">
         <material>Gazebo/Red</material>
         <sensor name="laser" type="ray">
@@ -77,4 +47,4 @@
             </plugin>
         </sensor>
-    </gazebo-->
+    </gazebo>
 </robot>
