Commit message: add lift to rls2_control and edit lidar

File: urdf/lift.xacro (robot description, xacro)
@@ -1,8 +1,9 @@
 <?xml version="1.0"?>
 <robot xmlns:xacro="http://www.ros.org/wiki/xacro">
+  <!-- Define properties -->
   <xacro:property name="screw_diameter" value="0.008" />
   <xacro:property name="screw_length" value="0.10" />
   <xacro:property name="plate_radius" value="0.045" />
-  <xacro:property name="screw_length" value="0.10" />
+  <!-- Link for the platform mid -->
   <link name="link_platform_mid">
     <origin xyz="0 0 0.0" rpy="0 0 0"/>
@@ -12,5 +13,5 @@
       </geometry>
       <material name="black">
-          <color rgba="0.1 0.1 0.1 1" />
+        <color rgba="0.1 0.1 0.1 1" />
       </material>
     </visual>
@@ -22,15 +23,16 @@
     <inertial>
       <mass value="1"/>
-      <inertia
-              ixx="1.0" ixy="0.0" ixz="0.0"
-              iyy="1.0" iyz="0.0"
-              izz="1.0"/>
+      <inertia ixx="1.0" ixy="0.0" ixz="0.0"
+               iyy="1.0" iyz="0.0"
+               izz="1.0"/>
     </inertial>
   </link>
+  <!-- Joint connecting upper link to platform mid -->
   <joint name="platform_joint" type="fixed">
     <parent link="upper_link" />
     <child link="link_platform_mid" />
-    <origin xyz="0.0 0 0.02" rpy="0. 0. 0."/>
+    <origin xyz="0.0 0 0.02" rpy="0 0 0"/>
   </joint>
+  <!-- Link for the lift mechanism -->
   <link name="lift_link">
     <visual>
@@ -45,21 +47,21 @@
     <collision>
       <geometry>
-         <mesh filename="package://robitcubebot_description/meshes/upperstand.STL" scale="0.001 0.001 0.001" />
+        <mesh filename="package://robitcubebot_description/meshes/upperstand.STL" scale="0.001 0.001 0.001" />
       </geometry>
     </collision>
     <inertial>
       <mass value="1"/>
-      <inertia
-              ixx="1.0" ixy="0.0" ixz="0.0"
-              iyy="1.0" iyz="0.0"
-              izz="1.0"/>
+      <inertia ixx="1.0" ixy="0.0" ixz="0.0"
+               iyy="1.0" iyz="0.0"
+               izz="1.0"/>
     </inertial>
   </link>
-  <joint name="lift_joint" type="prismatic" >
-    <origin xyz="0 0 0.08" rpy="0. 0. 0."/>
+  <!-- Prismatic joint for lifting -->
+  <joint name="lift_joint" type="prismatic">
+    <origin xyz="0 0 0.03" rpy="0 0 0"/>
+    <parent link="link_platform_mid" />
     <child link="lift_link" />
-    <parent link="link_platform_mid" />
     <axis xyz="0 0 1" rpy="0 0 0"/>
-    <limit effort="10000.0" lower="-0.05" upper="-0.035" velocity="0.2"/>
+    <limit effort="10000.0" lower="-0.05" upper="0.035" velocity="0.2"/>
     <dynamics damping="0.1" friction="0.1"/>
     <hardwareInterface>hardware_interface/VelocityJointInterface</hardwareInterface>

File: urdf/robitcubebot_ros2_control.xacro (robot description, xacro)
@@ -49,10 +49,9 @@
         </joint>
         <joint name="lift_joint">
-            <command_interface name="velocity">
-              <param name="min">-1</param>
-              <param name="max">1</param>
+            <command_interface name="position">
+            <param name="min">-05</param>
+            <param name="max">1.5</param>
             </command_interface>
-            <state_interface name="position" />
-            <state_interface name="velocity" />
+            <state_interface name="position"/>
         </joint>
     </ros2_control>
